File: DRV8300_4_LAYER_VQFN-24/DRV8300_4_LAYER.kicad_pcb (KiCad board)
At the start: 4 copper layers, 80.4 x 40.3 mm, 104 parts, among them Q1 SiR696DP, Q10 SiR696DP, Q11 SiR696DP, Q12 SiR696DP, Q13 SiR696DP, Q14 SiR696DP, Q15 SiR696DP, Q16 SiR696DP, Q17 SiR696DP, Q18 SiR696DP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

Commit message: VQFN-24
Parts:
- moved D3 22.7 mm to (193.7, 55.6)
- moved C20 21.8 mm to (200.6, 59.5), turned to 135 degrees
- moved D2 21.3 mm to (196.3, 56.5), turned to 90 degrees
- moved D1 19.3 mm to (198.1, 56.5), turned to 90 degrees
- moved U5 16.0 mm to (175.6, 57.2)
- moved C10 5.92 mm to (195.4, 51.6), turned to 180 degrees
- moved R25 3.65 mm to (190.2, 53.3)
- moved Q11 1.94 mm to (179.4, 65.9)
- moved Q19 1.94 mm to (187.0, 65.9)
- moved Q2 1.94 mm to (164.1, 65.9)
- moved Q5 1.94 mm to (171.7, 65.9)
- moved R1 1.94 mm to (190.9, 68.0)
- moved R2 1.94 mm to (183.2, 68.0)
- moved R5 1.94 mm to (175.6, 68.0)
- moved R6 1.94 mm to (167.9, 68.0)
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Routing:
- net +12V: track 1.89 -> 31.9 mm
- net /GHC: track 23.1 -> 51.2 mm, vias 4 -> 5
- net /GHA: track 24.4 -> 49.7 mm, vias 4 -> 5
- net /GHB: track 45.9 -> 23.7 mm, vias 4 -> 2
- net Net-(D3-K): track 0.00 -> 9.15 mm
- net Net-(D2-K): track 0.00 -> 4.97 mm
- net /MOTOR_B: track 97.4 -> 102.1 mm, vias 0 -> 1
- net Net-(Q21-G): track 4.42 -> 1.78 mm

Commit message: SAVE 19/04/26
Parts:
- C19: footprint Capacitor_SMD:C_0402_1005Metric -> Capacitor_SMD:C_0603_1608Metric
- moved C22 30.8 mm to (192.7, 64.0), turned to -90 degrees
- moved C21 23.5 mm to (197.0, 59.2), turned to 180 degrees
- moved C10 3.43 mm to (198.0, 53.8), turned to 0 degrees
- moved C19 1.97 mm to (197.8, 51.7), turned to 0 degrees
- moved D3 1.71 mm to (195.2, 56.6), turned to 90 degrees
- moved D1 0.88 mm to (198.9, 56.6)
- moved R18 0.79 mm to (223.2, 68.6)
- moved D2 0.74 mm to (197.1, 56.6)
- moved C20 0.66 mm to (201.1, 59.0), turned to 90 degrees
Routing:
- net /GHB: track 23.7 -> 69.5 mm, vias 2 -> 5
- net Net-(D1-K): track 0.00 -> 10.1 mm
- net +12V: track 31.9 -> 41.4 mm
- net /MOTOR_A: track 104.9 -> 110.1 mm
- net /MOTOR_C: track 94.1 -> 97.8 mm, vias 24 -> 25
- net /MOTOR_B: track 102.1 -> 105.7 mm, vias 1 -> 2
- net Net-(D3-K): track 9.15 -> 10.7 mm
- net /GHC: track 51.2 -> 51.8 mm
- net GND: vias 12 -> 25
