File: DRV8300_4_LAYER_VQFN-24/DRV8300_4_LAYER.kicad_sch (KiCad schematic)
At the start: 104 parts, among them Q1 SiR696DP, Q10 SiR696DP, Q11 SiR696DP, Q12 SiR696DP, Q13 SiR696DP, Q14 SiR696DP, Q15 SiR696DP, Q16 SiR696DP, Q17 SiR696DP, Q18 SiR696DP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

Commit message: SAVE 19/04/26
Parts:
- C19: footprint Capacitor_SMD:C_0402_1005Metric -> Capacitor_SMD:C_0603_1608Metric
Changed lines of the file:
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@@
 			)
 		)
-		(property "Footprint" "Capacitor_SMD:C_0402_1005Metric"
+		(property "Footprint" "Capacitor_SMD:C_0603_1608Metric"
 			(at 112.7252 41.91 0)
 			(effects
